Commit message: feat[robot]: combined all launches, new packages

File: src/moonlab_robots/urdf/robot.urdf.xacro (robot description, xacro)
@@ -3,11 +3,10 @@
     <xacro:include filename="$(find oakd_ros)/xacro/oakd.xacro" />
     <xacro:arg name="config_path" default="" />
-    <xacro:arg name="robot_name" default="kombai" />
-    <xacro:property name="all_mounts" value="${xacro.load_yaml('$(arg config_path)')}" />
-    <xacro:property name="data" value="${all_mounts['$(arg robot_name)']}" />
+    <xacro:arg name="robot_name" default="moonlab_robot" />
+    <xacro:property name="data" value="${xacro.load_yaml('$(arg config_path)')}" />
     <link name="base_link" />
     <xacro:oakd_camera
         parent_link="base_link"
-        xyz="${data['xyz'][0]} ${data['xyz'][1]} ${data['xyz'][2]}"
-        rpy="${data['rpy'][0]} ${data['rpy'][1]} ${data['rpy'][2]}" />
+        xyz="${data['x']} ${data['y']} ${data['z']}"
+        rpy="${data['roll']} ${data['pitch']} ${data['yaw']}" />
 </robot>
